Commit message: have a map but the robot drifts

File: src/mark1_description/urdf/mobile_base.xacro (robot description, xacro)
@@ -12,10 +12,11 @@
     <xacro:property name="gap_for_wheels" value="0.05" />
     <xacro:property name="gap_for_caster_wheels" value="${wheel_radius - (2*caster_wheel_radius)}" />
-    <!-- <link name="base_footprint">
-        <inertial>
-            <mass value="0.0001"/>
-            <inertia ixx="0.0001" ixy="0" ixz="0" iyy="0.0001" iyz="0" izz="0.0001"/>
-        </inertial>
-    </link> -->
+    <link name="base_footprint">
+    </link>
+    <joint name="base_footprint_base_link_joint" type="fixed">
+        <parent link="base_footprint"/>
+        <child link="base_link"/>
+        <origin xyz="0 0 ${base_height/2}" rpy="0 0 0"/>
+    </joint>
     <link name="base_link">
         <visual>

Commit message: fixed the wheels algined ground issue and, rtabmap.bd

File: src/mark1_description/urdf/mobile_base.xacro (robot description, xacro)
@@ -5,7 +5,7 @@
     <xacro:property name="base_height" value="0.6" />
     <xacro:property name="wheel_radius" value="0.1" />
-    <xacro:property name="wheel_length" value="0.05" />
+    <xacro:property name="wheel_width" value="0.05" />
     <xacro:property name="caster_wheel_radius" value="0.04" />
-    <xacro:property name="caster_wheel_length" value="0.025" />
+    <xacro:property name="caster_wheel_width" value="0.025" />
     <xacro:property name="pole_length" value="0.6" />
     <xacro:property name="pole_radius" value="0.02" />
@@ -14,8 +14,8 @@
     <link name="base_footprint">
     </link>
-    <joint name="base_footprint_base_link_joint" type="fixed">
+    <joint name="base_joint" type="fixed">
         <parent link="base_footprint"/>
         <child link="base_link"/>
-        <origin xyz="0 0 ${base_height/2}" rpy="0 0 0"/>
+        <origin xyz="0 0 ${wheel_radius}" rpy="0 0 0"/>
     </joint>
     <link name="base_link">
@@ -34,5 +34,5 @@
         </collision>
         <xacro:box_inertia m="20" x="${base_length}" y="${base_width}" z="${base_height}"
-                           o_xyz="0 0 ${base_height/2}" o_rpy="0 0 0" />
+                           o_xyz="0 0 0" o_rpy="0 0 0" />
     </link>
     <link name="pole_link">
@@ -57,5 +57,5 @@
             <visual>
                 <geometry>
-                    <cylinder radius="${wheel_radius}" length="${wheel_length}"/>
+                    <cylinder radius="${wheel_radius}" length="${wheel_width}"/>
                 </geometry>
                 <origin xyz="0 0 0" rpy="${pi/2.0} 0 0"/>
@@ -64,10 +64,10 @@
             <collision>
                 <geometry>
-                    <!--<cylinder radius="${wheel_radius}" length="${wheel_length}"/>-->
+                    <!--<cylinder radius="${wheel_radius}" length="${wheel_width}"/>-->
                     <sphere radius="${wheel_radius}" />
                 </geometry>
                 <origin xyz = "0 0 0" rpy="${pi/2.0} 0 0" />
             </collision>
-            <xacro:wheel_inertia m="0.2" r="${wheel_radius}" h="${wheel_length}"
+            <xacro:wheel_inertia m="0.2" r="${wheel_radius}" h="${wheel_width}"
                            o_xyz="0 0 0" o_rpy="${pi/2.0} 0 0" />
         </link>
@@ -79,5 +79,5 @@
             <visual>
                 <geometry>
-                    <cylinder radius="${caster_wheel_radius}" length="${caster_wheel_length}"/>
+                    <cylinder radius="${caster_wheel_radius}" length="${caster_wheel_width}"/>
                 </geometry>
                 <origin xyz="0 0 0" rpy="${pi/2.0} 0 0"/>
@@ -86,9 +86,9 @@
             <collision>
                 <geometry>
-                    <cylinder radius="${caster_wheel_radius}" length="${caster_wheel_length}"/>
+                    <cylinder radius="${caster_wheel_radius}" length="${caster_wheel_width}"/>
                 </geometry>
                 <origin xyz="0 0 0" rpy="${pi/2.0} 0 0"/>
             </collision>
-            <xacro:wheel_inertia m="0.05" r="${caster_wheel_radius}" h="${caster_wheel_length}"
+            <xacro:wheel_inertia m="0.05" r="${caster_wheel_radius}" h="${caster_wheel_width}"
                            o_xyz="0 0 0" o_rpy="${pi/2.0} 0 0" />
         </link>
@@ -110,15 +110,15 @@
         <parent link="base_link"/>
         <child link="front_left_wheel_link"/>
-        <origin xyz="${(base_length/4) + (2*caster_wheel_radius)} ${(base_width/2)-(caster_wheel_length/2)} ${-(caster_wheel_radius+gap_for_caster_wheels)}" rpy="0 0 0"/>
+        <origin xyz="${(base_length/4) + (2*caster_wheel_radius)} ${(base_width/2)-(caster_wheel_width/2)} ${-(caster_wheel_radius+gap_for_caster_wheels)}" rpy="0 0 0"/>
     </joint>
     <joint name="front_right_caster_joint" type="fixed">
         <parent link="base_link"/>
         <child link="front_right_wheel_link"/>
-        <origin xyz="${(base_length/4) + (2*caster_wheel_radius)} ${-((base_width/2)-(caster_wheel_length/2))} ${-(caster_wheel_radius+gap_for_caster_wheels)}" rpy="0 0 0"/>
+        <origin xyz="${(base_length/4) + (2*caster_wheel_radius)} ${-((base_width/2)-(caster_wheel_width/2))} ${-(caster_wheel_radius+gap_for_caster_wheels)}" rpy="0 0 0"/>
     </joint>
     <!--<joint name="base_front_right_wheel_joint" type="continuous">
         <parent link="base_link"/>
         <child link="front_right_wheel_link"/>
-        <origin xyz="${base_length/4} ${-((base_width/2)+(wheel_length/2))} 0" rpy="0 0 0"/>
+        <origin xyz="${base_length/4} ${-((base_width/2)+(wheel_width/2))} 0" rpy="0 0 0"/>
         <axis xyz="0 1 0"/>
     </joint>
@@ -126,5 +126,5 @@
         <parent link="base_link"/>
         <child link="front_left_wheel_link"/>
-        <origin xyz="${base_length/4} ${(base_width/2)+(wheel_length/2)} 0" rpy="0 0 0"/>
+        <origin xyz="${base_length/4} ${(base_width/2)+(wheel_width/2)} 0" rpy="0 0 0"/>
         <axis xyz="0 1 0"/>
     </joint>-->
@@ -132,5 +132,5 @@
         <parent link="base_link"/>
         <child link="rear_left_wheel_link"/>
-        <origin xyz="${-base_length/4} ${(base_width/2)+(wheel_length/2) + gap_for_wheels} 0" rpy="0 0 0"/>
+        <origin xyz="${-base_length/4} ${(base_width/2)+(wheel_width/2) + gap_for_wheels} 0" rpy="0 0 0"/>
         <axis xyz="0 1 0"/>
     </joint>
@@ -138,5 +138,5 @@
         <parent link="base_link"/>
         <child link="rear_right_wheel_link"/>
-        <origin xyz="${-base_length/4} ${-((base_width/2)+(wheel_length/2)+gap_for_wheels)} 0" rpy="0 0 0"/>
+        <origin xyz="${-base_length/4} ${-((base_width/2)+(wheel_width/2)+gap_for_wheels)} 0" rpy="0 0 0"/>
         <axis xyz="0 1 0"/>
     </joint>
